File: ctvt-pmod.kicad_sch (KiCad schematic)
At the start: 0 parts

Commit message: Complete routed CTVT energy monitor PMOD
Implement the ADS131M02 CT/VT analog front end, exact field connectors, chained PMOD interface, reproducible routing and branded fabrication-ready layout. Add architecture, calibration, safety documentation and final board renders.

Co-authored-by: Copilot <223556219+Copilot@users.noreply.github.com>
Parts:
- added C1, C2: 10nF C0G, Capacitor_SMD:C_0603_1608Metric, symbol ctvt-pmod-cache:C
- added C3, C5: 1uF, Capacitor_SMD:C_0603_1608Metric, symbol ctvt-pmod-cache:C
- added C4, C6: 100nF, Capacitor_SMD:C_0603_1608Metric, symbol ctvt-pmod-cache:C
- added C7: 220nF, Capacitor_SMD:C_0603_1608Metric, symbol ctvt-pmod-cache:C
- added D1: SMF3.3CA, Diode_SMD:D_SOD-123F, symbol ctvt-pmod-cache:TVS
- added D2: SMBJ18CA, Diode_SMD:D_SMB, symbol ctvt-pmod-cache:TVS
- added FB1: 600R@100MHz, Inductor_SMD:L_0603_1608Metric, symbol ctvt-pmod-cache:FB
- added J1: Tiny Tapeout PMOD, Connector_PinHeader_2.54mm:PinHeader_2x06_P2.54mm_Horizontal, symbol ctvt-pmod-cache:PMOD
- added J2: SJ-3523-SMT-TR, Connector_Audio:Jack_3.5mm_CUI_SJ-3523-SMT_Horizontal, symbol ctvt-pmod-cache:AUDIO_JACK
- added J3: PJ-002BH-SMT-TR, ctvt-pmod:DC_BARREL_JACK_SMD_2MM, symbol ctvt-pmod-cache:BARREL_JACK
- added J4: 613012243121, ctvt-pmod:PinSocket_2x06_P2.54mm_PMODHost1A, symbol ctvt-pmod-cache:PMOD_PASSIVE
- added R1, R2: 6.49R 0.1%, Resistor_SMD:R_0805_2012Metric, symbol ctvt-pmod-cache:R
- added R10, R3, R4, R9: 1k 0.1%, Resistor_SMD:R_0603_1608Metric, symbol ctvt-pmod-cache:R
- added R11, R12: 10k, Resistor_SMD:R_0603_1608Metric, symbol ctvt-pmod-cache:R
- added R13: 33R, Resistor_SMD:R_0603_1608Metric, symbol ctvt-pmod-cache:R
- added R5, R6: 100k 0.1%, Resistor_SMD:R_0805_2012Metric, symbol ctvt-pmod-cache:R
- added R7, R8: 6.49k 0.1%, Resistor_SMD:R_0805_2012Metric, symbol ctvt-pmod-cache:R
- added TP1: AIN0P, TestPoint:TestPoint_Pad_D1.0mm, symbol ctvt-pmod-cache:TP
- added TP2: AIN0N, TestPoint:TestPoint_Pad_D1.0mm, symbol ctvt-pmod-cache:TP
- added TP3: AIN1P, TestPoint:TestPoint_Pad_D1.0mm, symbol ctvt-pmod-cache:TP
- added TP4: AIN1N, TestPoint:TestPoint_Pad_D1.0mm, symbol ctvt-pmod-cache:TP
- added TP5: DRDY, TestPoint:TestPoint_Pad_D1.0mm, symbol ctvt-pmod-cache:TP
- added TP6: +3V3, TestPoint:TestPoint_Pad_D1.0mm, symbol ctvt-pmod-cache:TP
- added TP7: GND, TestPoint:TestPoint_Pad_D1.0mm, symbol ctvt-pmod-cache:TP
- added U1: ADS131M02IPWR, Package_SO:TSSOP-20_4.4x6.5mm_P0.65mm, symbol ctvt-pmod-cache:ADS131M02PW
Connections:
- new net +3V3: C5.1, C6.1, FB1.1, J1.12 (+3V3), J1.6 (+3V3), J4.12 (+3V3), J4.6 (+3V3), R11.1, R12.1, TP6.1, U1.20 (DVDD)
- new net AIN0N: C1.2, R4.2, TP2.1, U1.4 (AIN0N)
- new net AIN0P: C1.1, R3.2, TP1.1, U1.3 (AIN0P)
- new net AIN1N: C2.2, R10.2, TP4.1, U1.5 (AIN1N)
- new net AIN1P: C2.1, R9.2, TP3.1, U1.6 (AIN1P)
- new net AVDD: C3.1, C4.1, FB1.2, U1.1 (AVDD)
- new net CAP: C7.1, U1.18 (CAP)
- new net CLKIN: R13.2, U1.17 (CLKIN)
- new net CLK_HOST: J1.9 (CLKIN), J4.9 (CLKIN), R13.1
- new net CS: J1.1 (CS), J4.1 (CS), R11.2, U1.12 (~{CS})
- new net CT_N: D1.2, J2.S, R2.1, R4.1
- new net CT_P: D1.1, J2.T, R1.1, R3.1
- new net DRDY: J1.7 (DRDY), J4.7 (DRDY), TP5.1, U1.13 (~{DRDY})
- new net GND: C3.2, C4.2, C5.2, C6.2, C7.2, J1.11 (GND), J1.5 (GND), J2.R, J4.11 (GND), J4.5 (GND), R1.2, R2.2, R7.2, R8.2, TP7.1, U1.19 (DGND), U1.2 (AGND)
- new net MISO: J1.3 (MISO), J4.3 (MISO), U1.15 (DOUT)
- new net MOSI: J1.2 (MOSI), J4.2 (MOSI), U1.16 (DIN)
- new net RESERVED: J1.10 (RESERVED), J4.10 (RESERVED)
- new net RESET: J1.8 (RESET), J4.8 (RESET), R12.2, U1.11 (~{RESET})
- new net SCLK: J1.4 (SCLK), J4.4 (SCLK), U1.14 (SCLK)
- new net VT_DIV_N: R10.1, R6.2, R8.1
- new net VT_DIV_P: R5.2, R7.1, R9.1
- new net VT_N: D2.2, J3.2 (SLEEVE), R6.1
- new net VT_P: D2.1, J3.1 (CENTER), R5.1
- no-connect marks 0 -> 7
Other:
- note added: "CT INPUT - 100 A : 50 mA CT, 12.98 ohm split burden"
- note added: "POWER / DECOUPLING"
- note added: "SAFETY: ISOLATED CT AND CERTIFIED ISOLATED AC-AC TRANSFORMER ONLY. NEVER CONNECT MAINS DIRECTLY."
- note added: "TINY TAPEOUT PMOD"
- note added: "VT INPUT - isolated 9-12 VAC transformer only"
- company: (none) -> Whatnick
- title: (none) -> CTVT Energy Monitor PMOD

Commit message: Add sourced DigiKey bill of materials
Co-authored-by: Copilot <223556219+Copilot@users.noreply.github.com>
Parts:
- C1, C2: DigiKey PN (none) -> 490-9666-1-ND; MPN GRM1555C1H103JA01D -> GRM1885C1H103JA01D
- C3, C5: DigiKey PN (none) -> 399-C0603C105K4RACTUCT-ND; MPN (none) -> C0603C105K4RACTU; Manufacturer (none) -> KEMET
- C4, C6: DigiKey PN (none) -> 399-C0603C104K5RACTUCT-ND; MPN (none) -> C0603C104K5RACTU; Manufacturer (none) -> KEMET
- C7: DigiKey PN (none) -> 399-C0603C224K4RACTUCT-ND; MPN (none) -> C0603C224K4RACTU; Manufacturer (none) -> KEMET
- D1: DigiKey PN (none) -> 4786-GSMF3.3CACT-ND; MPN (none) -> GSMF3.3CA; Manufacturer (none) -> Good-Ark Semiconductor
- D2: DigiKey PN (none) -> SMBJ18CALFCT-ND; MPN (none) -> SMBJ18CA; Manufacturer (none) -> Littelfuse
- FB1: DigiKey PN (none) -> 445-MPZ1608S601ATA00CT-ND; MPN BLM15AG601SN1D -> MPZ1608S601ATA00; Manufacturer Murata -> TDK
- J1: DigiKey PN (none) -> 612-TSW-106-08-G-D-RA-ND; MPN (none) -> TSW-106-08-G-D-RA; Manufacturer (none) -> Samtec
- J2: DigiKey PN (none) -> CP-3523SJCT-ND
- J3: DigiKey PN (none) -> CP-002BHPJCT-ND
- J4: DigiKey PN (none) -> 732-613012243121-ND
- R10, R3, R4, R9: DigiKey PN (none) -> RG16P1.0KBCT-ND; MPN (none) -> RG1608P-102-B-T5; Manufacturer (none) -> Susumu
- R11, R12: DigiKey PN (none) -> RMCF0603FT10K0CT-ND; MPN (none) -> RMCF0603FT10K0; Manufacturer (none) -> Stackpole Electronics
- R13: DigiKey PN (none) -> 13-RC0603FR-0733RLCT-ND; MPN (none) -> RC0603FR-0733RL; Manufacturer (none) -> Yageo
- R5, R6: DigiKey PN (none) -> P100KDACT-ND; MPN (none) -> ERA-6AEB104V; Manufacturer (none) -> Panasonic Industry
- R7, R8: DigiKey PN (none) -> YAG1965CT-ND; MPN (none) -> RT0805BRD076K49L; Manufacturer (none) -> Yageo
- U1: DigiKey PN (none) -> 296-ADS131M02IPWRCT-ND

Commit message: Use TE precision burden resistors
Co-authored-by: Copilot <223556219+Copilot@users.noreply.github.com>
Parts:
- R1, R2: MPN TNPW08056R49BEEA -> RN73C2A6R49BTDF; Manufacturer Vishay -> TE Connectivity Holsworthy; Supplier (none) -> Mouser
Changed lines of the file:
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@@
 			)
 		)
-		(property "Manufacturer" "Vishay"
+		(property "Manufacturer" "TE Connectivity Holsworthy"
 			(at 76.2 46.99 0)
 			(effects
@@
 			)
 		)
-		(property "MPN" "TNPW08056R49BEEA"
+		(property "MPN" "RN73C2A6R49BTDF"
 			(at 76.2 46.99 0)
 			(effects
@@
 			)
 		)
-		(property "Description" "CT split burden resistor, 25 ppm/K; source outside DigiKey"
+		(property "Supplier" "Mouser"
+			(at 76.2 46.99 0)
+			(effects
+				(font
+					(size 1.27 1.27)
+				)
+				(hide yes)
+			)
+		)
+		(property "Description" "CT split burden resistor, 10 ppm/K"
 			(at 76.2 46.99 0)
 			(effects
@@
 			)
 		)
-		(property "Manufacturer" "Vishay"
+		(property "Manufacturer" "TE Connectivity Holsworthy"
 			(at 76.2 54.61 0)
 			(effects
@@
 			)
 		)
-		(property "MPN" "TNPW08056R49BEEA"
+		(property "MPN" "RN73C2A6R49BTDF"
 			(at 76.2 54.61 0)
 			(effects
@@
 			)
 		)
-		(property "Description" "CT split burden resistor, 25 ppm/K; source outside DigiKey"
+		(property "Supplier" "Mouser"
 			(at 76.2 54.61 0)
 			(effects
+				(font
+					(size 1.27 1.27)
+				)
+				(hide yes)
+			)
+		)
+		(property "Description" "CT split burden resistor, 10 ppm/K"
+			(at 76.2 54.61 0)
+			(effects

Commit message: Prepare Elecrow PCBA manufacturing package
Correct J4 to the vertical Wurth 61301221821 socket, add deterministic KiCad 10 manufacturing exports, and include verified Gerber, BOM, position, and combined Elecrow upload archives.

Co-authored-by: Copilot <223556219+Copilot@users.noreply.github.com>
Parts:
- J4: value 613012243121 -> 61301221821; DigiKey PN 732-613012243121-ND -> 732-61301221821-ND; MPN 613012243121 -> 61301221821
Changed lines of the file:
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@@
 			)
 		)
-		(property "Value" "613012243121"
+		(property "Value" "61301221821"
 			(at 248.92 154.94 0)
 			(effects
@@
 			)
 		)
-		(property "MPN" "613012243121"
+		(property "MPN" "61301221821"
 			(at 248.92 157.48 0)
 			(effects
@@
 			)
 		)
-		(property "DigiKey PN" "732-613012243121-ND"
+		(property "DigiKey PN" "732-61301221821-ND"
 			(at 248.92 157.48 0)
 			(effects
